File: kicad/prelab/prelab.kicad_sch (KiCad schematic)
At the start: 28 parts, among them M2 Motor, SW1 SW_Push, U1 PIC32MX170F256B, U2 SN754410, U3 USB2Serial, U4 Quadrature_Encoder

Commit message: Complete prelab kicad schematic
Parts:
- added C6: 0.1uF, symbol me218_library:Cap
- added R10, R11, R12, R5, R6, R7, R8, R9: 150, symbol me218_library:Res1
- added U5: 74HCT244, symbol 74xx:74HCT244
- BAR1: value HDSP-4830_2 -> LTA-1000HR
Connections:
- net +5V: now also C6.1, U5.20 (VCC)
- net GND: now also C6.2, R10.2, R11.2, R12.2, R5.2, R6.2, R7.2, R8.2, R9.2, U5.1 (1OE), U5.10 (GND), U5.19 (2OE)
- net at BAR1.10 (A): now also U5.9 (2Y3)
- net at BAR1.11 (K): now also R5.1
- net at BAR1.12 (K): now also R6.1
- net at BAR1.13 (K): now also R7.1
- net at BAR1.14 (K): now also R8.1
- net at BAR1.15 (K): now also R9.1
- net at BAR1.16 (K): now also R10.1
- net at BAR1.17 (K): now also R11.1
- net at BAR1.18 (K): now also R12.1
- net at BAR1.3 (A): now also U5.18 (1Y0)
- net at BAR1.4 (A): now also U5.16 (1Y1)
- net at BAR1.5 (A): now also U5.14 (1Y2)
- net at BAR1.6 (A): now also U5.12 (1Y3)
- net at BAR1.7 (A): now also U5.3 (2Y0)
- net at BAR1.8 (A): now also U5.5 (2Y1)
- net at BAR1.9 (A): now also U5.7 (2Y2)
- net at U2.10 (3A): no longer U1.21 (PGEC2/5VT/RB10)
- net at U2.15 (4A): no longer U1.22 (RB11)
Other:
- note added: "74HCT244"
- note added: "Enables for second motor"
- note added: "IC2"
- note added: "RA1"
- note added: "RA2"
- note added: "RA3"
- note added: "RA4"
- note added: "RB10"
- note added: "RB11"
- note added: "RB15"
- note added: "RB8"
- note added: "TO 74HCT244"
- note added: "VCC2 SN754410"
- note removed: "VCC2"
- company: (none) -> Stanford
- title: (none) -> ME218B lab 6 prelab 
- moved on the sheet: BAR1, C1, C2, C3, C4, C5, D1, D10, D2, D3, D4, D5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
